File: 0013_Joystick_Module_SKRHAAE010.kicad_sch (KiCad schematic)
At the start: 12 parts

Commit message: Add files via upload
Parts:
- added D1: LED, LED_SMD:LED_0805_2012Metric, symbol Device:LED
- added R11: R, Resistor_SMD:R_0805_2012Metric, symbol Device:R
- added U1: ~, Moduler_:pin_header, symbol moduler_pin:air
- R1, R10, R2, R3, R4, R5, R6, R7, R8, R9: footprint (none) -> Resistor_SMD:R_0805_2012Metric
- S1, S2: footprint SKRHAAE010 -> SKRHAAE010:SKRHAAE010
Connections:
- net +3V3: now also R11.1, U1.8
- net GND: now also D1.1 (K), U1.9
- net GPIO1: now also U1.1
- net GPIO10: now also U1.14
- net GPIO2: now also U1.2
- net GPIO3: now also U1.3
- net GPIO4: now also U1.4
- net GPIO5: now also U1.5
- net GPIO6: now also U1.18
- net GPIO7: now also U1.17
- net GPIO8: now also U1.16
- net GPIO9: now also U1.15
- new net: D1.2 (A), R11.2
- no-connect marks 0 -> 6
Other:
- moved on the sheet: R1, R10, R2, R3, R4, R5, R6, R7, R8, R9, S1, S2
